Commit message: init commit

File: nav2-slam-navigation/docker/src/navigation2/nav2_system_tests/urdf/turtlebot3_burger.urdf (robot description, URDF)
Before this commit: robot turtlebot3_burger, 7 links, 6 joints
Links:
- removed link base_footprint
Joints:
- joint base_joint: parent base_footprint -> base_link

File: nav2-slam-navigation/docker/src/navigation2/nav2_system_tests/urdf/turtlebot3_waffle.urdf (robot description, URDF)
Before this commit: robot turtlebot3_waffle, 13 links, 12 joints
Links:
- removed link base_footprint
Joints:
- joint base_joint: parent base_footprint -> base_link
